File: pedal-pcb/Seed.kicad_sch (KiCad schematic)
At the start: 42 parts, among them J1 In L, J10 FS1, J11 OutR, J2 Power, J3 In R, J4 SW1, J5 OutL, J6 LEDs, J7 Pot1, J8 Pot2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

Commit message: Update PCB to KiCad 8
Other:
- company: (none) -> MA&I
- title: (none) -> Daisy Seed, Stereo Inputs & Outputs
